File: MCM51A_Repro/MCM51A_Repro.kicad_sch (KiCad schematic)
At the start: 38 parts, among them J1 Conn_01x04, J2 Conn_02x25_Odd_Even, P1 DE9_Receptacle_MountingHoles, U1 80C31, U2 74LS373, U3 27C020, U4 27C020, U5 GAL16V8, U6 MAX232, Y1 Crystal

Commit message: Adding comments to annotated equations, and condensing schematic to a single (legal) sheet)
Parts:
- P1: value DE9_Receptacle_MountingHoles -> DE9 Receptacle
- U4: value 27C020 -> RAM
Other:
- moved on the sheet: C1, C10, C11, C12, C13, C14, C15, C2, C3, C4, C5, C6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
